File: Lamps/v2/v2.1.0/LampDriver.kicad_pcb (KiCad board)
At the start: 2 copper layers, 50 x 42.8 mm, 24 parts, among them J1 JST XH 1x4, J2 Screw_Terminal_01x02, J3 1x6 MOLEX KK 396, Q1 BSS138, Q2 BSS138, Q3 BSS138, Q4 TSM7P06CP, Q5 TSM7P06CP, Q6 TSM7P06CP

Commit message: First draft of hardware docs
Signed-off-by: Patrick Pedersen <ctx.xda@gmail.com>
Other:
- board text added: "Jukebox Lamp Driver Rev 2.1.0"
- board text removed: "Jukebox Lamp Driver Rev 2.0.0"
