File: Lamps/v2/v2.1.0/LampDriver.kicad_sch (KiCad schematic)
At the start: 27 parts, among them J1 JST XH 1x4, J2 Screw_Terminal_01x02, J3 1x6 MOLEX KK 396, Q1 BSS138, Q2 BSS138, Q3 BSS138, Q4 FDD4141, Q5 FDD4141, Q6 FDD4141

Commit message: First draft of hardware docs
Signed-off-by: Patrick Pedersen <ctx.xda@gmail.com>
Other:
- note added: "Rev 2.1.0 - Patrick Pedersen <ctx.xda@gmail.com>"
- note removed: "Rev 2.0.0 - Patrick Pedersen <ctx.xda@gmail.com>"
Changed lines of the file:
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@@
 (kicad_sch
-	(version 20231120)
+	(version 20250114)
 	(generator "eeschema")
-	(generator_version "8.0")
+	(generator_version "9.0")
 	(paper "A4")
 	(title_block
@@
 		(company "TuDo Makerspace")
 	)
+	(rectangle
+		(start 162.56 77.47)
+		(end 231.14 110.49)
+		(stroke
+			(width 0)
+			(type dash_dot)
+		)
+		(fill
+			(type none)
+		)
+	)
+	(rectangle
+		(start 166.37 120.65)
+		(end 232.41 130.81)
+		(stroke
+			(width 0)
+			(type dash)
+		)
+		(fill
+			(type none)
+		)
+	)
+	(text "Input/Output follows direct logic.\nIn other words:\n\n	3.3V INPUT -> LIGHT ON\n	0V   INPUT -> LIGHT OFF"
+		(exclude_from_sim no)
+		(at 18.796 160.02 0)
+		(effects
+			(font
+				(size 1.27 1.27)
+			)
+			(justify left)
+		)
+	)
+	(text "Jukebox Lamps"
+		(exclude_from_sim no)
+		(at 252.476 87.63 0)
+		(effects
+			(font
+				(size 1.27 1.27)
+			)
+		)
+	)
+	(text "MOLEX"
+		(exclude_from_sim no)
+		(at 229.362 119.38 0)
+		(effects
+			(font
+				(size 1.27 1.27)
+			)
+		)
+	)
+	(text "Rev 2.1.0 - Patrick Pedersen <ctx.xda@gmail.com>"
+		(exclude_from_sim no)
+		(at 17.78 30.226 0)
+		(effects
+			(font
+				(size 5.08 5.08)
+			)
+			(justify left)
+		)
+	)
+	(text "Input/Low Side (3.3V)"
+		(exclude_from_sim no)
+		(at 81.788 53.086 0)
+		(effects
+			(font
+				(size 3.81 3.81)
+				(thickness 0.762)
+				(bold yes)
+			)
+		)
+	)
+	(text "! HEATSINK MAY BE REQUIRED !"
+		(exclude_from_sim no)
+		(at 235.458 113.03 0)
+		(effects
+			(font
+				(size 1.27 1.27)
+			)
+		)
+	)
+	(text "github.com/TuDo-Makerspace"
+		(exclude_from_sim no)
+		(at 17.78 39.37 0)
+		(effects
+			(font
+				(size 2.54 2.54)
+			)
+			(justify left)
+		)
+	)
+	(text "Output/High Side (12V)"
+		(exclude_from_sim no)
+		(at 217.678 52.832 0)
+		(effects
+			(font
+				(size 3.81 3.81)
+				(thickness 0.762)
+				(bold yes)
+			)
+		)
+	)
+	(text "RPi GPIO's"
+		(exclude_from_sim no)
+		(at 21.336 112.268 0)
+		(effects
+			(font
+				(size 1.27 1.27)
+			)
+		)
+	)
+	(text "TuDo Makerspace Jukebox: Lamp Driver Board"
+		(exclude_from_sim no)
+		(at 16.51 19.05 0)
+		(effects
+			(font
+				(size 6.35 6.35)
+				(thickness 1.27)
+				(bold yes)
+			)
+			(justify left)
+		)
+	)
 	(junction
 		(at 41.91 66.04)
@@
 		)
 	)
-	(rectangle
-		(start 162.56 77.47)
-		(end 231.14 110.49)
-		(stroke
-			(width 0)
-			(type dash_dot)
-		)
-		(fill
-			(type none)
-		)
-	)
-	(rectangle
-		(start 166.37 120.65)
-		(end 232.41 130.81)
-		(stroke
-			(width 0)
-			(type dash)
-		)
-		(fill
-			(type none)
-		)
-	)
-	(text "Input/Output follows direct logic.\nIn other words:\n\n	3.3V INPUT -> LIGHT ON\n	0V   INPUT -> LIGHT OFF"
-		(exclude_from_sim no)
-		(at 18.796 160.02 0)
-		(effects
-			(font
-				(size 1.27 1.27)
-			)
-			(justify left)
-		)
-	)
-	(text "Jukebox Lamps"
-		(exclude_from_sim no)
-		(at 252.476 87.63 0)
-		(effects
-			(font
-				(size 1.27 1.27)
-			)
-		)
-	)
-	(text "MOLEX"
-		(exclude_from_sim no)
-		(at 229.362 119.38 0)
-		(effects
-			(font
-				(size 1.27 1.27)
-			)
-		)
-	)
-	(text "Rev 2.0.0 - Patrick Pedersen <ctx.xda@gmail.com>"
-		(exclude_from_sim no)
-		(at 17.78 30.226 0)
-		(effects
-			(font
-				(size 5.08 5.08)
-			)
-			(justify left)
-		)
-	)
-	(text "Input/Low Side (3.3V)"
-		(exclude_from_sim no)
-		(at 81.788 53.086 0)
-		(effects
-			(font
-				(size 3.81 3.81)
-				(thickness 0.762)
-				(bold yes)
-			)
-		)
-	)
-	(text "! HEATSINK MAY BE REQUIRED !"
-		(exclude_from_sim no)
-		(at 235.458 113.03 0)
-		(effects
-			(font
-				(size 1.27 1.27)
-			)
-		)
-	)
-	(text "github.com/TuDo-Makerspace"
-		(exclude_from_sim no)
-		(at 17.78 39.37 0)
-		(effects
-			(font
-				(size 2.54 2.54)
-			)
-			(justify left)
-		)
-	)
-	(text "Output/High Side (12V)"
-		(exclude_from_sim no)
-		(at 217.678 52.832 0)
-		(effects
-			(font
-				(size 3.81 3.81)
-				(thickness 0.762)
-				(bold yes)
-			)
-		)
-	)
-	(text "RPi GPIO's"
-		(exclude_from_sim no)
-		(at 21.336 112.268 0)
-		(effects
-			(font
-				(size 1.27 1.27)
-			)
-		)
-	)
-	(text "TuDo Makerspace Jukebox: Lamp Driver Board"
-		(exclude_from_sim no)
-		(at 16.51 19.05 0)
-		(effects
-			(font
-				(size 6.35 6.35)
-				(thickness 1.27)
-				(bold yes)
-			)
-			(justify left)
-		)
-	)
 	(label "L1+"
 		(at 242.57 69.85 0)
@@
 		)
 	)
+	(embedded_fonts no)
 )
