File: Keypad/Keypad.kicad_sch (KiCad schematic)
At the start: 34 parts, among them Q1 PNP, Q2 PNP, SW1 SW_Push, SW10 SW_Push, SW11 SW_Push, SW12 SW_Push, SW13 SW_Push, SW14 SW_Push, SW15 SW_Push, SW16 SW_Push, SW2 SW_Push, SW3 SW_Push, SW4 SW_Push, SW5 SW_Push, SW6 SW_Push, SW7 SW_Push, SW8 SW_Push, SW9 SW_Push

Commit message: Keypad: Kicad schematic completed
Signed-off-by: Patrick Pedersen <ctx.xda@gmail.com>
Parts:
- removed SW1: SW_Push, symbol Switch:SW_Push
- added D1, D2: 3.3V, symbol Device:D_Zener
- SW10: value SW_Push -> 2
- SW11: value SW_Push -> 8
- SW12: value SW_Push -> 0
- SW13: value SW_Push -> 4
- SW14: value SW_Push -> 1
- SW15: value SW_Push -> 7
- SW16: value SW_Push -> R
- SW5: value SW_Push -> 6
- SW6: value SW_Push -> 3
- SW7: value SW_Push -> 9
- SW8: value SW_Push -> G
- SW9: value SW_Push -> 5
- renumbered SW4 to BLUE, D3 to D401, D4 to D402, D5 to D403, D6 to D404, D2 to D405, D1 to D406, R1 to R401, R2 to R402, R3 to R403, R4 to R404, SW3 to RED, Q1 to T401, Q2 to T403, SW2 to YELLOW
Connections:
- net GND: now also D1.2 (A), D2.2 (A)
- net 2: now reaches R5.1, T401.1 (C)
- net at D405.1 (K), D406.1 (K), SW13.1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: now also SW16.2; no longer SW16.1
- net 1: now reaches R6.1, T403.1 (C)
- net A renamed GPIO24
- net B renamed GPIO23
- net C renamed 3
- net 3: now also D2.1 (K)
- net D renamed 4
- net 4: now also D1.1 (K)
- new net: D402.2 (A), D403.2 (A), RED.2, SW11.2, SW15.2, SW7.2
- new net: BLUE.1, R401.2, R402.2, R403.2, RED.1, T401.3 (E), T403.3 (E), YELLOW.1
- new net: BLUE.2, D404.2 (A), SW12.2, SW16.1, SW8.2
- new net: D401.2 (A), SW10.2, SW14.2, SW6.2, YELLOW.2
- new net: R404.1, SW13.2, SW5.2, SW9.2
- no-connect marks 0 -> 2
Other:
- note added: "Decoder (On RPi Perfboard)"
- note added: "Keypad PCB"
- note added: "Seperate PCB"
- moved on the sheet: D401, D402, D403, D404, D405, D406, R10, R401, R402, R403, R404, R5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

Commit message: Docs: More keypad stuff
Signed-off-by: Patrick Pedersen <ctx.xda@gmail.com>
Parts:
- D401, D402, D403, D404, D405, D406: value D -> 1N4148
Changed lines of the file:
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@@
 	)
 	(junction
-		(at 111.76 162.56)
+		(at 111.76 168.91)
 		(diameter 0)
 		(color 0 0 0 0)
@@
 	)
 	(junction
-		(at 27.94 163.83)
+		(at 27.94 170.18)
 		(diameter 0)
 		(color 0 0 0 0)
@@
 	)
 	(junction
-		(at 74.93 163.83)
+		(at 74.93 170.18)
 		(diameter 0)
 		(color 0 0 0 0)
@@
 	)
 	(junction
-		(at 137.16 162.56)
+		(at 137.16 168.91)
 		(diameter 0)
 		(color 0 0 0 0)
@@
 	)
 	(junction
-		(at 52.07 163.83)
+		(at 52.07 170.18)
 		(diameter 0)
 		(color 0 0 0 0)
@@
 	(wire
 		(pts
-			(xy 137.16 162.56) (xy 137.16 190.5)
+			(xy 137.16 168.91) (xy 137.16 190.5)
 		)
 		(stroke
@@
 	(wire
 		(pts
-			(xy 27.94 151.13) (xy 27.94 163.83)
+			(xy 27.94 151.13) (xy 27.94 170.18)
 		)
 		(stroke
@@
 	(wire
 		(pts
-			(xy 137.16 109.22) (xy 137.16 162.56)
+			(xy 137.16 109.22) (xy 137.16 168.91)
 		)
 		(stroke
@@
 	(wire
 		(pts
-			(xy 27.94 163.83) (xy 31.75 163.83)
+			(xy 27.94 170.18) (xy 31.75 170.18)
 		)
 		(stroke
@@
 	(wire
 		(pts
-			(xy 74.93 163.83) (xy 78.74 163.83)
+			(xy 74.93 170.18) (xy 78.74 170.18)
 		)
 		(stroke
@@
 	(wire
 		(pts
-			(xy 52.07 154.94) (xy 52.07 163.83)
+			(xy 52.07 154.94) (xy 52.07 170.18)
 		)
 		(stroke
@@
 	(wire
 		(pts
-			(xy 137.16 162.56) (xy 140.97 162.56)
+			(xy 137.16 168.91) (xy 140.97 168.91)
 		)
 		(stroke
@@
 	(wire
 		(pts
-			(xy 111.76 162.56) (xy 115.57 162.56)
+			(xy 111.76 168.91) (xy 115.57 168.91)
 		)
 		(stroke
@@
 	(wire
 		(pts
-			(xy 27.94 163.83) (xy 27.94 237.49)
+			(xy 27.94 170.18) (xy 27.94 237.49)
 		)
 		(stroke
@@
 	(wire
 		(pts
-			(xy 111.76 162.56) (xy 111.76 190.5)
+			(xy 111.76 168.91) (xy 111.76 190.5)
 		)
 		(stroke
@@
 	(wire
 		(pts
-			(xy 52.07 163.83) (xy 55.88 163.83)
+			(xy 52.07 170.18) (xy 55.88 170.18)
 		)
 		(stroke
@@
 	(wire
 		(pts
-			(xy 111.76 91.44) (xy 111.76 162.56)
+			(xy 111.76 91.44) (xy 111.76 168.91)
 		)
 		(stroke
@@
 	(wire
 		(pts
-			(xy 74.93 154.94) (xy 74.93 163.83)
+			(xy 74.93 154.94) (xy 74.93 170.18)
 		)
 		(stroke
@@
 	(wire
 		(pts
-			(xy 52.07 163.83) (xy 52.07 215.9)
+			(xy 52.07 170.18) (xy 52.07 215.9)
 		)
 		(stroke
@@
 	(wire
 		(pts
-			(xy 74.93 163.83) (xy 74.93 210.82)
+			(xy 74.93 170.18) (xy 74.93 210.82)
 		)
 		(stroke
@@
 	)
 	(label "4"
-		(at 55.88 163.83 0)
+		(at 55.88 170.18 0)
 		(effects
 			(font
@@
 	)
 	(label "2"
-		(at 115.57 162.56 0)
+		(at 115.57 168.91 0)
 		(effects
 			(font
@@
 	)
 	(label "6 (GND)"
-		(at 31.75 163.83 0)
+		(at 31.75 170.18 0)
 		(effects
 			(font
@@
 	)
 	(label "1"
-		(at 140.97 162.56 0)
+		(at 140.97 168.91 0)
 		(effects
 			(font
@@
 	)
 	(label "3"
-		(at 78.74 163.83 0)
+		(at 78.74 170.18 0)
 		(effects
 			(font
@@
 			)
 		)
-		(property "Value" "D"
+		(property "Value" "1N4148"
 			(at 71.12 148.5899 90)
 			(effects
@@
 			)
 		)
-		(property "Value" "D"
+		(property "Value" "1N4148"
 			(at 127 114.2999 90)
 			(effects
@@
 			)
 		)
-		(property "Value" "D"
+		(property "Value" "1N4148"
 			(at 43.18 148.5899 90)
 			(effects
@@
 			)
 		)
-		(property "Value" "D"
+		(property "Value" "1N4148"
 			(at 55.88 148.5899 90)
 			(effects
@@
 			)
 		)
-		(property "Value" "D"
+		(property "Value" "1N4148"
 			(at 83.82 148.5899 90)
 			(effects
@@
 			)
 		)
-		(property "Value" "D"
+		(property "Value" "1N4148"
 			(at 101.6 113.0299 90)
 			(effects
