File: Lamps/v2/v2.2.1/LampDriver.kicad_sch (KiCad schematic)
At the start: 28 parts, among them J1 JST XH 1x4, J2 Screw_Terminal_01x02, J3 1x6 MOLEX KK 396, Q1 BSS138, Q2 BSS138, Q3 BSS138, Q4 FDD4141, Q5 FDD4141, Q6 FDD4141

Commit message: Lamps: PCB: minor changes qualify as v2.2.1
Signed-off-by: Patrick Pedersen <ctx.xda@gmail.com>
Other:
- note added: "Rev 2.2.1 - Patrick Pedersen <ctx.xda@gmail.com>"
- note removed: "Rev 2.2.0 - Patrick Pedersen <ctx.xda@gmail.com>"
Changed lines of the file:
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@@
 		)
 	)
-	(text "Rev 2.2.0 - Patrick Pedersen <ctx.xda@gmail.com>"
+	(text "Rev 2.2.1 - Patrick Pedersen <ctx.xda@gmail.com>"
 		(exclude_from_sim no)
 		(at 17.78 30.226 0)
